File: 16550.sch (KiCad schematic (older format))
At the start: 5 parts, among them J16 DSUB-9, U13 PAL16L8, U14 74AHC1G04, U15 16550, U16 max235cpg

Commit message: update 16650
Parts:
- added C? (x2): 0.1uF, symbol Device:C
Connections:
- net GND: now also C?.1, C?.1
- net VCC: now also C?.2, C?.2
Changed lines of the file:
@@
 L power:VCC #PWR08
 U 1 1 60EE6A9F
-P 5900 1550
-F 0 "#PWR08" H 5900 1400 50  0001 C CNN
-F 1 "VCC" H 5915 1723 50  0000 C CNN
-F 2 "" H 5900 1550 50  0001 C CNN
-F 3 "" H 5900 1550 50  0001 C CNN
-	1    5900 1550
-	1    0    0    -1
+P 6150 1550
+F 0 "#PWR08" H 6150 1400 50  0001 C CNN
+F 1 "VCC" V 6165 1678 50  0000 L CNN
+F 2 "" H 6150 1550 50  0001 C CNN
+F 3 "" H 6150 1550 50  0001 C CNN
+	1    6150 1550
+	0    1    1    0
 $EndComp
 NoConn ~ 4900 4450
 Wire Wire Line
+	5900 1550 6150 1550
+Wire Wire Line
+	6150 1550 6150 1400
+Connection ~ 6150 1550
+$Comp
+L Device:C C?
+U 1 1 60F65FED
+P 6150 1250
+F 0 "C?" H 6265 1296 50  0000 L CNN
+F 1 "0.1uF" H 6265 1205 50  0000 L CNN
+F 2 "" H 6188 1100 50  0001 C CNN
+F 3 "~" H 6150 1250 50  0001 C CNN
+	1    6150 1250
+	1    0    0    -1
+$EndComp
+$Comp
+L power:GND #PWR?
+U 1 1 60F66904
+P 6150 1100
+F 0 "#PWR?" H 6150 850 50  0001 C CNN
+F 1 "GND" H 6155 927 50  0000 C CNN
+F 2 "" H 6150 1100 50  0001 C CNN
+F 3 "" H 6150 1100 50  0001 C CNN
+	1    6150 1100
+	-1   0    0    1
+$EndComp
+$Comp
+L power:VCC #PWR?
+U 1 1 60F6AFA9
+P 8050 1400
+F 0 "#PWR?" H 8050 1250 50  0001 C CNN
+F 1 "VCC" V 8065 1528 50  0000 L CNN
+F 2 "" H 8050 1400 50  0001 C CNN
+F 3 "" H 8050 1400 50  0001 C CNN
+	1    8050 1400
+	0    1    1    0
+$EndComp
+Wire Wire Line
+	7800 1400 8050 1400
+Wire Wire Line
+	8050 1400 8050 1250
+Connection ~ 8050 1400
+$Comp
+L Device:C C?
+U 1 1 60F6AFB2
+P 8050 1100
+F 0 "C?" H 8165 1146 50  0000 L CNN
+F 1 "0.1uF" H 8165 1055 50  0000 L CNN
+F 2 "" H 8088 950 50  0001 C CNN
+F 3 "~" H 8050 1100 50  0001 C CNN
+	1    8050 1100
+	1    0    0    -1
+$EndComp
+$Comp
+L power:GND #PWR?
+U 1 1 60F6AFB8
+P 8050 950
+F 0 "#PWR?" H 8050 700 50  0001 C CNN
+F 1 "GND" H 8055 777 50  0000 C CNN
+F 2 "" H 8050 950 50  0001 C CNN
+F 3 "" H 8050 950 50  0001 C CNN
+	1    8050 950
+	-1   0    0    1
+$EndComp
+Wire Wire Line
 	3200 3250 3350 3250
